File: firefly-instruments/firefly-instrument-tray.brd (EAGLE design)
At the start: 220 x 100 mm, 117 parts, among them J1 CON-26, J2 USB-4PINUSB-B1HSB6, J3 CON-220020303-D021B01LF, J4 CON-26, J5 CON-26, J6 CON-10SWD, J7 CON-10SWD, U10 PTC0603, U1:C1 1uF, U1:J1 SMFLP, U1:R1 10k, U1:R2 4.7k, U1:R3 4.7k, U1:U1 TCS3471, U2:Q1 FET-NSOT-23-3, U2:U1 TXS2SA, U3:Q1 FET-NSOT-23-3, U3:U1 TXS2SA, U4:Q1 FET-NSOT-23-3, U4:U1 TXS2SA, U5:Q1 FET-NSOT-23-3, U5:U1 TXS2SA, U6:Q1 FET-NSOT-23-3, U6:U1 74LVCH1T45, U6:U2 74LVCH1T45, U7:Q1 FET-NSOT-23-3, U7:U1 74LVCH1T45, U7:U2 74LVCH1T45, U8:C1 1nF, U8:C2 100nF, U8:C3 10uF, U8:C4 1nF, U8:C7 1uF, U8:C9 100nF, U8:L1 1k, U8:L2 1k, U8:R1 1.8K, U8:R16 1, U8:R2 0, U8:R3 43, U8:R4 12K, U8:R5 10k, U8:R6 10k, U8:R7 376, U8:R8 1K, U8:U1 LTC6102-1MS8, U8:U2 TLV272, U9:C1 4700uF, U9:C10 1nF, U9:C11 100nF, U9:C12 10uF, U9:C13 1nF, U9:C14 1nF, U9:C15 100nF, U9:C16 1nF, U9:C17 1uF, U9:C18 100nF, U9:C19 100nF, U9:C2 100nF, U9:C3 100nF, U9:C4 1uF, U9:C5 1uF, U9:C7 4.7uF, U9:C8 510pF, U9:D1 D-US, U9:L1 22uH, U9:L2 1k, U9:L3 1k, U9:Q1 FET-NSOT-23-3, U9:R1 1K, U9:R10 200 (2W WW), U9:R11 650K, U9:R12 100K, U9:R13 100K, U9:R15 36K, U9:R16 396K, U9:R18 1.8K, U9:R19 0, U9:R2 10K, U9:R20 43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

Commit message: instrument tray ready to fab first version
Parts:
- removed J3: CON-220020303-D021B01LF, firefly:20020303-D021B01LF
- removed U$4: FRDM-K22F, firefly:FRDM-K22F
- removed U1:R2, U1:R3: 4.7k, firefly:R0603
- added C1, C12, C13, C15, C2, C3: 100nF, firefly:C0805
- added C10, C11: 1uF, firefly:C0805
- added C14: 10uF, firefly:C0805
- added C4: 1uF, firefly:C0603
- added C5, C6: 22pF, firefly:C0805
- added C7, C8: 4.7uF, firefly:C0805
- added C9: 10nF, firefly:C0805
- added D1: LED-RGB-CAMSL0201RGB, firefly:MSL0201RGB
- added J10: CON-2WC-2, firefly:WC-2
- added J8: USB-4PINUSB-B1HSB6, firefly:USB-B1HSB6
- added J9: CON-10SWD, firefly:SWD-10
- added R10, R16: 60, firefly:R0805
- added R11, R9: 22, firefly:R0805
- added R12: 72.5k, firefly:R0805
- added R13: 10K, firefly:R0805
- added R14, R15: 4.7k, firefly:R0603
- added R17: 240, firefly:R0805
- added R19: 0, firefly:R0805
- added R7, R8: 1k, firefly:R0603
- added U11:Q1: FET-NSOT-23-3, firefly:SOT-23-3
- added U11:U1: TXS2SA, firefly:TXS2SA
- added U12: AP7331, firefly:SOT-23-5
- added U13: MCP47X6, firefly:SOT-23-6
- added U14: STM32F411-LQFP64, firefly:LQFP-64
- added X1: XTAL2TXC_7A, firefly:TXC_7A
- U9:C3: device firefly:C3216 -> firefly:C0805
- U9:L1: device firefly:L2012C -> firefly:L3225P
- moved U9:L2 11.3 mm to (104.2, 31.2)
- moved U9:L3 11.3 mm to (119.6, 31.2)
- moved U9:C11 11.2 mm to (104.3, 25.0)
- moved U9:C12 11.2 mm to (106.8, 25.0)
- moved U9:C13 11.2 mm to (111.0, 18.5)
- moved U9:C14 11.2 mm to (116.8, 14.4)
- moved U9:C15 11.2 mm to (104.4, 12.0)
- moved U9:C16 11.2 mm to (111.0, 5.00)
- moved U9:C17 11.2 mm to (122.3, 25.0)
- moved U9:C18 11.2 mm to (110.8, 11.4)
- moved U9:C19 11.2 mm to (110.9, 25.0)
- moved U9:R18 11.2 mm to (95.8, 29.3)
- moved U9:R19 11.2 mm to (106.8, 29.3)
- moved U9:R20 11.2 mm to (100.2, 29.3)
- moved U9:R22 11.2 mm to (110.9, 20.9)
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Connections:
- removed net ATE_LCS_SCL: J5.7, U$4.J2.20, U1:R3.1, U1:U1.2
- removed net ATE_LCS_SDA: J5.9, U$4.J2.18, U1:R2.1, U1:U1.6
- removed net P3V3_1: U$4.J25.8
- removed net P5-9V_IN: U$4.J25.16
- removed net P5V_USB: U$4.J25.10
- new net ATE_BATTERY+2: J5.12, R7.2, R8.1, U14.25
- new net ATE_BATTERY+_SENSE: J5.8, U11:Q1.1, U14.51
- new net ATE_SCL: J5.7, R15.1, U13.5, U14.61, U1:U1.2
- new net ATE_SDA: J5.9, R14.1, U13.4, U14.59, U1:U1.6
- new net BOOT0: R19.1, U14.60
- new net N$1: R10.2, U14.2
- new net N$10: C8.1, U14.30
- new net N$11: R12.1, R13.2, U12.4
- new net N$12: J8.2, R11.2
- new net N$13: R17.2, U14.4
- new net N$14: J8.3, R9.2
- new net N$15: D1.3, R10.1
- new net N$16: D1.1, R16.1
- new net N$17: D1.2, R17.1
- new net N$18: J10.1, U14.16
- new net N$4: R7.1, U11:U1.5
- new net N$5: C5.1, U14.6, X1.2
- new net N$6: C6.1, U14.5, X1.1
- new net N$7: R16.2, U14.3
- new net NRESET: J9.10, U14.7
- new net SWCLK: J9.4, U14.49
- new net SWDIO: J9.2, U14.46
- new net U11:ANC: U11:U1.3
- new net U11:BC: U11:U1.9
- new net U11:BNC: U11:U1.10
- new net U11:BNO: U11:U1.8
- new net U11:N$2: U11:Q1.3, U11:U1.12
- new net USB_DM: R11.1, U14.44
- new net USB_DP: R9.1, U14.45
- new net USB_VBUS: C10.1, C7.1, J8.1, U12.1, U12.3, U14.42, U8:L1.1, U8:L2.1, U9:C4.1, U9:C7.1, U9:L1.1, U9:L2.1, U9:L3.1, U9:U2.1, U9:U3.5
- net +3V3: now also C1.1, C11.1, C13.1, C14.1, C15.1, C2.1, C3.1, C4.1, C9.1, D1.4, J9.1, R12.2, R14.2, R15.2, U11:U1.1, U12.5, U13.3, U14.1, U14.13, U14.19, U14.32, U14.48, U14.64; no longer U1:R2.2, U1:R3.2
- net +5V: now also J2.1; no longer J3.1A, J3.1B, J5.25, U8:L1.1, U8:L2.1, U9:C4.1, U9:C7.1, U9:L1.1, U9:L2.1, U9:L3.1, U9:U2.1, U9:U3.5
- net ATE_BS_ADJ: now also C12.1, U13.1; no longer U$4.J24.11
- net ATE_BS_EN: now also U14.52; no longer U$4.J2.8
- net ATE_BS_SHR: now also U14.20; no longer U$4.J24.1
- net ATE_BS_SLR: now also U14.21; no longer U$4.J24.5
- net ATE_BUTTON_EN: now also U14.53; no longer U$4.J2.10
- net ATE_MCU1_VCC2: now also U14.17; no longer U$4.J1.12
- net ATE_MCU2_VCC2: now also U14.23; no longer U$4.J1.6
- net ATE_MCU_VCC_SENSE: now also U14.54; no longer U$4.J2.12
- net ATE_SWD1_DIR_TO_DUT: now also U14.26; no longer U$4.J1.1
- net ATE_SWD1_NRESET: now also U14.27; no longer U$4.J1.3
- net ATE_SWD1_PWR: now also U14.29; no longer U$4.J1.7
- net ATE_SWD1_SWDCLK: now also U14.28; no longer U$4.J1.5
- net ATE_SWD1_SWDIO: now also U14.33; no longer U$4.J1.9
- net ATE_SWD2_DIR_TO_DUT: now also U14.37; no longer U$4.J1.14
- net ATE_SWD2_NRESET: now also U14.38; no longer U$4.J1.16
- net ATE_SWD2_PWR: now also U14.40; no longer U$4.J2.4
- net ATE_SWD2_SWDCLK: now also U14.39; no longer U$4.J2.2
- net ATE_SWD2_SWDIO: now also U14.41; no longer U$4.J2.6
- net ATE_USB_5V_EN: now also U14.34; no longer U$4.J1.11
- net ATE_USB_CS_EN: now also U14.35; no longer U$4.J1.13
- net ATE_USB_CS_OUT: now also U14.22; no longer U$4.J24.8
- net ATE_USB_D_EN: now also U14.36; no longer U$4.J1.15
- net DUT_BATTERY+: now also U11:U1.4
- net DUT_GND: now also J5.10, R8.2, U14.24
- net DUT_MCU2_BOOT0: now also U14.50; no longer U$4.J1.2
- net GND: now also C1.2, C10.2, C11.2, C12.2, C13.2, C14.2, C15.2, C2.2, C3.2, C4.2, C5.2, C6.2, C7.2, C8.2, C9.2, J10.2, J8.4, J9.3, J9.5, R13.1, R19.2, U11:Q1.2, U12.2, U13.2, U14.12, U14.18, U14.31, U14.47, U14.63; no longer J3.2A, J3.2B, U$4.J2.14, U$4.J25.12, U$4.J25.14
Routing:
- net USB_VBUS: track 0.00 -> 290.5 mm, vias 0 -> 8
- net +5V: track 309.0 -> 21.1 mm, vias 8 -> 2
- net ATE_SDA: track 0.00 -> 250.1 mm, vias 0 -> 7
- net ATE_SCL: track 0.00 -> 247.8 mm, vias 0 -> 4
- net ATE_BATTERY+_SENSE: track 0.00 -> 214.6 mm, vias 0 -> 5
- net ATE_BATTERY+2: track 0.00 -> 213.8 mm, vias 0 -> 5
- net +3V3: track 282.1 -> 495.8 mm, vias 2 -> 13
- net DUT_GND: track 400.8 -> 565.9 mm, vias 6 -> 10
- net ATE_LCS_SCL: track 128.3 -> 0.00 mm, vias 3 -> 0
- net DUT_BATTERY+: track 118.4 -> 243.8 mm, vias 1 -> 6
- net ATE_LCS_SDA: track 123.4 -> 0.00 mm, vias 5 -> 0
- net NRESET: track 0.00 -> 100.5 mm, vias 0 -> 4
- net DUT_MCU2_BOOT0: track 153.7 -> 204.8 mm, vias 1 -> 5
- net GND: track 80.9 -> 128.5 mm, vias 44 -> 64
- net N$17: track 0.00 -> 47.1 mm, vias 0 -> 2
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Other:
- board size 220 x 100 mm -> 193 x 100 mm
- board text added: "Firefly Instruments revision 0.1 2016/05/09 © Firefly Design LLC"

Commit message: rev 0.2 of instrument board
Parts:
- added J11, J12: CON-2282847-2, firefly:282847-2
- added J13, J14: CON-1CT3151, firefly:CT3151
- added U9:C6: 10uF, firefly:C0805
- C4, U1:C1: device firefly:C0603 -> firefly:C0805
- J10: value CON-2WC-2 -> CON-2CON-HEADER-2; device firefly:WC-2 -> firefly:CON-HEADER-2
- R1: device firefly:R0805 -> firefly:KRL6432
- R14, R15, R3, R4, R5, R6, R7, R8, U1:R1: device firefly:R0603 -> firefly:R0805
- R2: device firefly:R2010 -> firefly:RW0S6BB
- U11:Q1, U2:Q1, U3:Q1, U4:Q1, U5:Q1, U6:Q1, U7:Q1, U9:Q1: value FET-NSOT-23-3 -> FET-NMCPH3; device firefly:SOT-23-3 -> firefly:MCPH3
- U8:U2, U9:U6, U9:U8: value TLV272 -> TLV271SN2T1G
- U9:D1: value D-US -> D-USSOD-123A; device firefly:D0603 -> firefly:SOD-123A
- U9:R10, U9:R6: device firefly:R2512 -> firefly:RCL1225
- U9:R7, U9:R9: device firefly:R2512 -> firefly:KRL6432
- moved R2 22.9 mm to (72.0, 58.0), turned to 270 degrees
- moved U9:R4 8.68 mm to (112.0, 40.0), turned to 180 degrees
- moved U9:C14 7.28 mm to (111.0, 10.0)
- moved U9:C10 7.06 mm to (111.0, 23.6)
- moved J2 5.30 mm to (22.4, 89.5)
- moved R7 3.07 mm to (82.2, 29.0)
- moved R8 3.04 mm to (78.0, 29.0)
- moved R1 2.77 mm to (9.00, 61.5)
- moved U9:R3 2.60 mm to (122.1, 38.5)
- moved U9:Q1 2.40 mm to (122.2, 45.0)
- moved U9:R6 2.40 mm to (122.2, 54.4)
- moved U8:R1 1.90 mm to (5.80, 56.5)
- moved U9:R5 1.80 mm to (106.2, 38.6)
- moved U9:C18 1.61 mm to (111.0, 13.0)
- moved U9:C7 1.60 mm to (78.1, 38.6)
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Connections:
- removed net N$18: J10.1, U14.16
- new net EXP_PA2: J10.1, J12.1, U14.16
- net +5V: now also J13.1, J13.2, J13.3, J13.4
- net DUT_BUTTON+: now also J11.1
- net GND: now also J11.2, J12.2, J14.1, J14.2, J14.3, J14.4, U9:C6.2
- net U8:N$11: now also U8:U2.3; no longer U8:U2.4
- net U8:N$12: now also U8:U2.4; no longer U8:U2.3
- net U9:+12V: now also U9:C6.1
- net U9:N$19: now also U9:U6.3; no longer U9:U6.4
- net U9:N$20: now also U9:U6.4; no longer U9:U6.3
- net U9:N$26: now also U9:U8.3; no longer U9:U8.4
- net U9:N$27: now also U9:U8.4; no longer U9:U8.3
Routing:
- net DUT_BUTTON+: track 118.9 -> 249.3 mm, vias 3 -> 4
- net DUT_GND: track 565.9 -> 498.2 mm
- net ATE_BS_ADJ: track 153.6 -> 94.9 mm
- net DUT_MOTOR+: track 69.6 -> 37.2 mm
- net EXP_PA2: track 0.00 -> 27.5 mm
- net N$18: track 11.0 -> 0.00 mm
- net GND: track 128.5 -> 120.2 mm, vias 64 -> 66
- net N$22: track 89.2 -> 96.4 mm, vias 1 -> 2
- net N$21: track 104.4 -> 111.1 mm
- net N$3: track 23.1 -> 28.7 mm
- net U9:N$5: track 8.54 -> 3.96 mm, vias 2 -> 0
- net N$2: track 106.5 -> 110.9 mm
- net U8:VOA: track 18.0 -> 13.7 mm
- net N$4: track 23.9 -> 28.0 mm
- net U8:N$11: track 10.7 -> 14.7 mm
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Other:
- board text added: "Firefly Instruments Revision 0.2 2016/06/1 Copyright Firefly Design LLC"
- board text removed: "Firefly Instruments revision 0.1 2016/05/09 © Firefly Design LLC"
