File: firefly-instruments/firefly-instrument-tray.sch (EAGLE design)
At the start: 15 parts, among them J1 CON-26, J2 USB-4PINUSB-B1HSB6, J3 CON-220020303-D021B01LF, J4 CON-26, J5 CON-26, J6 CON-10SWD, J7 CON-10SWD, U10 PTC0603

Commit message: instrument tray ready to fab first version
Parts:
- removed J3: CON-220020303-D021B01LF, firefly:CON-220020303-D021B01LF
- removed U$4: FRDM-K22F, firefly:FRDM-K22F
- added C1, C12, C13, C15, C2, C3: 100nF, firefly:C-USC0805
- added C10, C11: 1uF, firefly:C-USC0805
- added C14: 10uF, firefly:C-USC0805
- added C4: 1uF, firefly:C-USC0603
- added C5, C6: 22pF, firefly:C-USC0805
- added C7, C8: 4.7uF, firefly:C-USC0805
- added C9: 10nF, firefly:C-USC0805
- added D1: LED-RGB-CAMSL0201RGB, firefly:LED-RGB-CAMSL0201RGB
- added J10: CON-2WC-2, firefly:CON-2WC-2
- added J8: USB-4PINUSB-B1HSB6, firefly:USB-4PINUSB-B1HSB6
- added J9: CON-10SWD, firefly:CON-10SWD
- added R10, R16: 60, firefly:R-USR0805
- added R11, R9: 22, firefly:R-USR0805
- added R12: 72.5k, firefly:R-USR0805
- added R13: 10K, firefly:R-USR0805
- added R14, R15: 4.7k, firefly:R-USR0603
- added R17: 240, firefly:R-USR0805
- added R19: 0, firefly:R-USR0805
- added R7, R8: 1k, firefly:R-USR0603
- added U12: AP7331, firefly:AP7331
- added U13: MCP47X6, firefly:MCP47X6
- added U14: STM32F411-LQFP64, firefly:STM32F411-LQFP64
- added X1: XTAL2TXC_7A, firefly:XTAL2TXC_7A
- J1, J4, J5: MANUFACTURER (none) -> Amphenol FCI; ORDERING-CODE (none) -> 68602-126HLF
- J2: MANUFACTURER (none) -> On Shore Technology Inc.; ORDERING-CODE (none) -> USB-B1HSB6
- J6, J7: MANUFACTURER (none) -> Harwin; ORDERING-CODE (none) -> M50-3500542
- R1: MANUFACTURER (none) -> Susumu; ORDERING-CODE (none) -> KRL6432E-M-R100-F-T1
- R3, R4, R5, R6: MANUFACTURER (none) -> Yageo; ORDERING-CODE (none) -> RC0805FR-0710KL
- U10: MANUFACTURER (none) -> Bel Fuse Inc.; ORDERING-CODE (none) -> 0ZCM0016FF2G
Connections:
- removed net ATE_LCS_SCL: J5.7, U$4.PTE1
- removed net ATE_LCS_SDA: J5.9, U$4.PTE0
- removed net SCL: R3.1
- removed net SDA: R2.1
- new net +12V: C8.1, D1.C, R16.2, R8.1
- new net ADJ: R13.1
- new net ATE_BATTERY+2: J5.12, R7.2, R8.1, U14.PC5
- new net ATE_BATTERY+_SENSE: J5.8, U14.PC10
- new net ATE_SCL: J5.7, R15.1, U13.SCL, U14.PB8
- new net ATE_SDA: J5.9, R14.1, U13.SDA, U14.PB7
- new net BOOT0: R19.1, U14.BOOT0
- new net N$12: D1.A, J8.D-, R11.2, R7.1, R8.1
- new net N$13: R17.2, R19.2, U14.PC15-OSC32_OUT
- new net N$14: C11.1, J8.D+, R9.2
- new net N$15: D1.B, R10.1
- new net N$16: D1.G, R16.1
- new net N$17: D1.R, R17.1
- new net N$18: C13.2, J10.1, U14.PA2
- new net N$19: C10.1
- new net N$26: C14.1
- new net N$6: C6.1, C8.2, R15.2, R16.1, U14.PH0-OSC_IN, X1.1
- new net NRESET: J9.10, U14.NRST
- new net SENSE: C4.1, R7.2
- new net SENSE_HIGH_RANGE: C13.1
- new net SWCLK: J9.4, U14.PA14
- new net SWDIO: J9.2, U14.PA13
- new net USB_DM: R11.1, U14.PA11
- new net USB_DP: R9.1, U14.PA12
- new net USB_VBUS: C10.1, C7.1, J8.5V, U12.EN, U12.IN, U14.PA9
- new net VOA: C7.1, C9.1, R16.1
- net +3V3: now also C1.1, C11.1, C13.1, C14.1, C15.1, C2.1, C3.1, C4.1, C9.1, D1.A, J9.1, R12.2, R14.2, R15.2, U12.OUT, U13.VDD, U14.VBAT, U14.VDD1, U14.VDD2, U14.VDD3, U14.VDD4, U14.VDDA/VREF+; no longer R2.2, R3.2
- net +5V: now also C4.1, C7.1, J2.5V; no longer J3.1, J5.25
- net ATE_BS_ADJ: now also C12.1, U13.VOUT; no longer U$4.DAC0_OUT
- net ATE_BS_EN: now also U14.PC11; no longer U$4.PTD6
- net ATE_BS_SHR: now also U14.PA4; no longer U$4.ADC0_DP0
- net ATE_BS_SLR: now also U14.PA5; no longer U$4.ADC0_DP3
- net ATE_BUTTON_EN: now also U14.PC12; no longer U$4.PTD7
- net ATE_MCU1_VCC2: now also U14.PA3; no longer U$4.PTB18
- net ATE_MCU2_VCC2: now also U14.PA7; no longer U$4.PTB16
- net ATE_MCU_VCC_SENSE: now also U14.PD2; no longer U$4.PTD5
- net ATE_SWD1_DIR_TO_DUT: now also U14.PB0; no longer U$4.PTA5
- net ATE_SWD1_NRESET: now also U14.PB1; no longer U$4.PTA13
- net ATE_SWD1_PWR: now also U14.PB10; no longer U$4.PTC8
- net ATE_SWD1_SWDCLK: now also U14.PB2; no longer U$4.PTA12
- net ATE_SWD1_SWDIO: now also U14.PB12; no longer U$4.PTC9
- net ATE_SWD2_DIR_TO_DUT: now also U14.PC6; no longer U$4.PTC3
- net ATE_SWD2_NRESET: now also U14.PC7; no longer U$4.PTC6
- net ATE_SWD2_PWR: now also U14.PC9; no longer U$4.PTA1
- net ATE_SWD2_SWDCLK: now also U14.PC8; no longer U$4.PTB19
- net ATE_SWD2_SWDIO: now also U14.PA8; no longer U$4.PTD4
- net ATE_USB_5V_EN: now also U14.PB13; no longer U$4.PTC7
- net ATE_USB_CS_EN: now also U14.PB14; no longer U$4.PTC10
- net ATE_USB_CS_OUT: now also U14.PA6; no longer U$4.PTC2
- net ATE_USB_D_EN: now also U14.PB15; no longer U$4.PTC5
- net BAT+: now also C5.1, R10.2, R11.2, R7.2
- net BAT-: now also C1.2, C2.2, R9.2
- net DUT_GND: now also J5.10, R8.2, U14.PC4
- net DUT_MCU2_BOOT0: now also U14.PA15; no longer U$4.PTD2
- net GND: now also C1.2, C10.2, C11.2, C12.2, C13.2, C14.2, C15.2, C2.2, C3.2, C4.2, C5.2, C6.2, C7.2, C8.2, C9.2, J10.2, J8.GND, J9.3, J9.5, R10.1, R12.1, R13.1, R15.1, R19.2, R8.2, R9.1, U12.GND, U13.VSS, U14.VSS1, U14.VSS2, U14.VSS3, U14.VSS4, U14.VSSA/VREF-; no longer J3.2, U$4.GND, U$4.GND1, U$4.GND2
- net N$1: now also R10.2, U14.PC13
- net N$10: now also C4.2, C8.1, U14.VCAP1
- net N$11: now also C1.1, R12.1, R13.2, U12.ADJ
- net N$2: now also R16.2
- net N$21: now also C15.1
- net N$3: now also C2.1, C3.1
- net N$4: now also R11.1, R12.2, R13.2, R7.1
- net N$5: now also C5.1, U14.PH1-OSC_OUT, X1.2
- net N$7: now also C2.1, R16.2, R8.2, U14.PC14-OSC32_IN
- net N$8: now also C3.2
- net N$9: now also C1.1, R7.1
- net VCSA: now also C11.2, C12.1, C15.2, C2.2, C3.1, R19.1
Other:
- note added: "DAC"
- note added: "VSS/VDD 1-4 Decoupling"
- note added: "VSSA/VDDA Decoupling"
- moved on the sheet: J1, J4, J5, R1, R2, U10

Commit message: rev 0.2 of instrument board
Parts:
- added J11, J12: CON-2282847-2, firefly:CON-2282847-2
- added J13, J14: CON-1CT3151, firefly:CON-1CT3151
- C4: device firefly:C-USC0603 -> firefly:C-USC0805
- C5, C6: MANUFACTURER AVX Corporation -> Samsung Electro-Mechanics America, Inc.; ORDERING-CODE SQCAEM220JAJME -> CL21C220FBANNNC
- J10: value CON-2WC-2 -> CON-2CON-HEADER-2; device firefly:CON-2WC-2 -> firefly:CON-2CON-HEADER-2
- R1: device firefly:R-USR0805 -> firefly:R-USKRL6432
- R14, R15, R3, R4, R5, R6, R7, R8: device firefly:R-USR0603 -> firefly:R-USR0805
- R2: device firefly:R-USR2010 -> firefly:R-USRW0S6BB
Connections:
- new net EXP_PA2: J10.1, J12.1, U14.PA2
- net +12V: now also C6.1
- net +5V: now also J13.1
- net DUT_BUTTON+: now also J11.1
- net GND: now also J11.2, J12.2, J14.1
- net N$18: no longer J10.1, U14.PA2
Other:
- note added: "add relay to connect battery simulator output to DUT battery+"
