File: firefly-instruments/firefly-instrument-tray.sch (EAGLE design)
At the start: 52 parts, among them J1 CON-26, J10 CON-2CON-HEADER-2, J11 CON-2282847-2, J12 CON-2282847-2, J13 CON-1CT3151, J14 CON-1CT3151, J2 USB-4PINUSB-B1HSB6, J4 CON-26, J5 CON-26, J6 CON-10SWD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

Commit message: Firefly Instrument Tray 0.3 (out for fab)
Parts:
- removed J10: CON-2CON-HEADER-2, firefly:CON-2CON-HEADER-2
- removed J11, J12: CON-2282847-2, firefly:CON-2282847-2
- removed J4, J5: CON-26, firefly:CON-26
- removed R8: 1k, firefly:R-USR0805
- added C16: 1F, firefly:C-USPM118
- added C17: 100nF, firefly:C-USC0805
- added J3: CON-4282847-4, firefly:CON-4282847-4
- added R18: 1 (2W WW), firefly:R-USRCL1225
- added R20: 49.9 (2W WW), firefly:R-USKRL6432
- added R21: 49.9 (2W WW), firefly:R-USRCL1225
- added U17: MEMORY-SPISOA008, firefly:MEMORY-SPISOA008
- J13: MANUFACTURER (none) -> B&K Precision; ORDERING-CODE (none) -> CT3151-2
- J14: MANUFACTURER (none) -> B&K Precision; ORDERING-CODE (none) -> CT3151-0
- R7: value 1k -> 10k
Connections:
- removed net +12V: C6.1, C8.1, D1.C, R16.2, R8.1
- removed net ATE_BATTERY+_SENSE: J5.8, U14.PC10
- removed net ATE_USB_D_EN: J4.25, U14.PB15
- removed net BAT-: C1.2, C2.2, R3.1, R5.1, R9.2
- removed net EXP_PA2: J10.1, J12.1, U14.PA2
- removed net N$22: J2.D-
- new net ATE_BAT_ADJ_EN: U14.PC10
- new net ATE_BAT_CAP_EN: U14.PB3
- new net ATE_DRAIN_EN: U14.PB5
- new net ATE_FILL_EN: U14.PB4
- new net ATE_SWD1_SENSE_NRESET: U14.PB6
- new net ATE_SWD2_SENSE_NRESET: U14.PB9
- new net BATCAP: R18.1
- new net DRAINCAP: R21.1
- new net DUT_NRESET: R2.2
- new net DUT_SWDCLK: R1.2
- new net DUT_SWDIO: R17.2
- new net DUT_SWITCH_1: J3.1
- new net DUT_SWITCH_2: J3.2
- new net EN: R13.2
- new net FILLCAP: R20.1
- new net MEM_CSN: R7.1, U14.PB15, U17.!CS
- new net N$25: C16.2
- new net SENSE_LOW_RANGE: C16.1
- new net SENSE_R: R18.2
- new net SENSE_S: R20.1
- new net SPI_MISO: U14.PA2, U17.DO
- new net SPI_MOSI: U14.PA1, U17.DI
- new net SPI_SCLK: U14.PA0, U17.CLK
- net +3V3: now also C17.1, R7.2, U17.!HOLD, U17.!WP, U17.VCC; no longer J5.26
- net +5V: no longer C7.1
- net ATE_BATTERY+2: no longer J5.12, R7.2, R8.1
- net ATE_BS_ADJ: no longer J5.2
- net ATE_BS_EN: no longer J4.1
- net ATE_BS_SHR: no longer J5.6
- net ATE_BS_SLR: no longer J5.4
- net ATE_BUTTON_EN: no longer J4.3
- net ATE_MCU1_VCC2: no longer J5.1
- net ATE_MCU2_VCC2: no longer J5.3
- net ATE_MCU_VCC_SENSE: no longer J4.5
- net ATE_SCL: no longer J5.7
- net ATE_SDA: no longer J5.9
- net ATE_SWD1_DIR_TO_DUT: no longer J4.7
- net ATE_SWD1_NRESET: no longer J4.9
- net ATE_SWD1_PWR: no longer J4.11
- net ATE_SWD1_SWDCLK: no longer J4.13
- net ATE_SWD1_SWDIO: no longer J4.17
- net ATE_SWD2_DIR_TO_DUT: no longer J4.8
- net ATE_SWD2_NRESET: no longer J4.10
- net ATE_SWD2_PWR: no longer J4.12
- net ATE_SWD2_SWDCLK: no longer J4.14
- net ATE_SWD2_SWDIO: no longer J4.18
- net ATE_USB_5V_EN: no longer J4.21
- net ATE_USB_CS_EN: no longer J4.23
- net ATE_USB_CS_OUT: no longer J5.5
- net BAT+: no longer R10.2, R6.2, R7.2
- net DUT_BUTTON+: no longer J11.1
- net DUT_GND: no longer J5.10, R8.2
- net DUT_I2C_DRDY: no longer J4.22
- net DUT_I2C_SCL: no longer J4.26
- net DUT_I2C_SDA: no longer J4.24
- net DUT_MCU2_BOOT0: no longer J4.20
- net DUT_SPI_MISO: no longer J4.6
- net DUT_SPI_MOSI: no longer J4.4
- net DUT_SPI_SCLK: no longer J4.2
- net DUT_USB_5V: now also J3.3
- net DUT_VB: no longer J4.16
- net GND: now also C16.2, C17.2, J3.4, R21.2, U17.GND; no longer J10.2, J11.2, J12.2, J4.15, J4.19, R10.1, R15.1, R4.1, R8.2, R9.1
- net N$1: now also R2.1; no longer R1.1
- net N$10: no longer R6.1
- net N$12: no longer D1.A, R8.1
- net N$15: now also R18.1
- net N$16: now also R20.2
- net N$17: now also R21.1
- net N$2: now also R17.1; no longer R3.2
- net N$21: no longer J2.D+
- net N$3: no longer C3.1, R2.1
- net N$4: now also C16.1, R18.2, R20.2, R21.2; no longer R7.1
- net N$5: no longer R4.2
- net N$6: no longer C8.2, R15.2, R16.1
- net N$7: no longer C2.1, R8.2
- net N$8: no longer C3.2, R5.2
- net N$9: no longer C1.1, R7.1
- net VOA: now also C17.1
Other:
- note added: "+"
- note added: "160 mA Hold 400 mA Trip"
- note removed: "12V Supply"
- note removed: "Button"
- note removed: "Current Shunt"
- note removed: "ESR"
- note removed: "NOTE: DUT GND can be above GND"
- note removed: "add relay to connect battery simulator output to DUT battery+"
- moved on the sheet: C10, C11, J2, J6, J7, R1, R12, R13, R14, R15, R2, R3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

Commit message: Rev 0.4 instrument board - ready for production
Connections:
- new net BAT-: R1.2
- net GND: now also R1.1
Changed lines of the file:
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@@
 <part name="Q1" library="firefly" deviceset="FET-N" device="MCPH3" value="FET-NMCPH3">
 <attribute name="MANUFACTURER" value="ON Semiconductor"/>
-<attribute name="ORDERING-CODE" value="MCH3484-TL-H"/>
+<attribute name="ORDERING-CODE" value="MCH3481-TL-W"/>
 </part>
 <part name="V1" library="firefly" deviceset="GND" device=""/>
@@
 <part name="Q1" library="firefly" deviceset="FET-N" device="MCPH3" value="FET-NMCPH3">
 <attribute name="MANUFACURER" value="ON Semiconductor"/>
-<attribute name="ORDERING-CODE" value="MCH3484-TL-H"/>
+<attribute name="ORDERING-CODE" value="MCH3481-TL-W"/>
 </part>
 <part name="V2" library="firefly" deviceset="GND" device=""/>
@@
 </part>
 <part name="V5" library="firefly" deviceset="GND" device=""/>
+<part name="R1" library="firefly" deviceset="R-US" device="R0805" value="0">
+<attribute name="MANUFACTURER" value="Yageo"/>
+<attribute name="ORDERING-CODE" value="RC0805FR-070RL"/>
+</part>
+<part name="V6" library="firefly" deviceset="GND" device=""/>
 </parts>
 <sheets>
@@
 </instance>
 <instance part="V5" gate="GND" x="33.02" y="109.22"/>
+<instance part="R1" gate="G$1" x="246.38" y="68.58">
+<attribute name="MANUFACTURER" x="246.38" y="68.58" size="1.778" layer="96" display="off"/>
+<attribute name="ORDERING-CODE" x="246.38" y="68.58" size="1.778" layer="96" display="off"/>
+</instance>
+<instance part="V6" gate="GND" x="238.76" y="63.5"/>
 </instances>
 <busses>
@@
 <wire x1="251.46" y1="68.58" x2="271.78" y2="68.58" width="0.1524" layer="91"/>
 <label x="266.7" y="68.58" size="1.778" layer="95"/>
+<pinref part="R1" gate="G$1" pin="2"/>
 </segment>
 </net>
@@
 <pinref part="U2" gate="G$1" pin="GND"/>
 <wire x1="58.42" y1="157.48" x2="58.42" y2="160.02" width="0.1524" layer="91"/>
+</segment>
+<segment>
+<pinref part="R1" gate="G$1" pin="1"/>
+<pinref part="V6" gate="GND" pin="GND"/>
+<wire x1="241.3" y1="68.58" x2="238.76" y2="68.58" width="0.1524" layer="91"/>
+<wire x1="238.76" y1="68.58" x2="238.76" y2="66.04" width="0.1524" layer="91"/>
 </segment>
 </net>
@@
 <net name="DUT_BATTERY+" class="0">
 <segment>
-<wire x1="48.26" y1="177.8" x2="68.58" y2="177.8" width="0.1524" layer="91"/>
-<label x="48.26" y="177.8" size="1.778" layer="95"/>
-</segment>
-<segment>
 <portref moduleinst="U15" port="BNO"/>
 <wire x1="134.62" y1="152.4" x2="144.78" y2="152.4" width="0.1524" layer="91"/>
@@
 <label x="243.84" y="40.64" size="1.778" layer="95"/>
 </segment>
-<segment>
-<wire x1="93.98" y1="177.8" x2="109.22" y2="177.8" width="0.1524" layer="91"/>
-<label x="93.98" y="177.8" size="1.778" layer="95"/>
-</segment>
-</net>
+</net>

Commit message: fix SPI memory ordering code
Parts:
- U17: ORDERING-CODE S25FL116K0XMFI013 -> S25FL116K0XMFI043
Changed lines of the file:
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@@
 <?xml version="1.0" encoding="utf-8"?>
 <!DOCTYPE eagle SYSTEM "eagle.dtd">
-<eagle version="7.5.0">
+<eagle version="7.7.0">
 <drawing>
 <settings>
@@
 <part name="U17" library="firefly" deviceset="MEMORY-SPI" device="SOA008" value="MEMORY-SPISOA008">
 <attribute name="MANUFACTURER" value="Cypress Semiconductor Corp"/>
-<attribute name="ORDERING-CODE" value="S25FL116K0XMFI013"/>
+<attribute name="ORDERING-CODE" value="S25FL116K0XMFI043"/>
 </part>
 <part name="+3V6" library="supply1" deviceset="+3V3" device=""/>

Commit message: add battery simulator voltage to A/D; separate motor minus from ground; remove J2; bump to version 0.5
Parts:
- removed J2: USB-4PINUSB-B1HSB6, firefly:USB-4PINUSB-B1HSB6
Connections:
- removed net BAT-: R1.2
- removed net DUT_GND: J1.23, J1.24, J1.25, J1.4, J6.3, J6.5, J7.3, J7.5, R2.2, U14.PC4
- new net DUT_MOTOR-: J1.25, R2.2
- new net N$35: R2.2
- new net SENSE_V2: R1.2, R2.1
- net +5V: no longer J2.5V
- net GND: now also J1.23, J1.24, J1.4, J6.3, J6.5, J7.3, J7.5; no longer J2.GND
Other:
- note removed: "!!! Calculate Rx For Max 4.3V"
- note removed: "Adjustable Voltage"

Commit message: revision 0.5 ready for production
Parts:
- C5, C6: MANUFACTURER Samsung Electro-Mechanics America, Inc. -> KEMET; ORDERING-CODE CL21C220FBANNNC -> C0805C220F5GACTU
- J14: ORDERING-CODE CT3151-0 -> CT3151SP-0
- U12: value AP7331 -> VREG-ADJAP7331-WG-7; device firefly:AP7331 -> firefly:VREG-ADJAP7331-WG-7
- X1: value XTAL2TXC_7A -> XTAL2CX5032GA; device firefly:XTAL2TXC_7A -> firefly:XTAL2CX5032GA; MANUFACTURER TXC CORPORATION -> AVX Corp/Kyocera Corp; ORDERING-CODE 7A-8.000MAAE-T -> CX5032GA08000H0PST02
Other:
- note added: "Module: BATTERY_SIMULATOR"
- note added: "Module: BATTERY_SIMULATOR (Page 1 of 2)"
- note added: "Module: BATTERY_SIMULATOR (Page 2 of 2)"
- note added: "Module: COLOR_SENSOR"
- note added: "Module: CURRENT_SENSE"
- note added: "Module: RELAY"
- note added: "Module: SERIAL_WIRE_DEBUG"
- note added: "Top Level"
- note removed: "USB"
- moved on the sheet: R3, R4, R5, R6
